File: PCB - EC Version/keyboard.kicad_pcb (KiCad board)
At the start: 2 copper layers, 286.4 x 103.6 mm, 123 parts, among them J1 HRO_TYPE-C-31-M-12, J2 Conn_01x03, SW1 Alps SKRK, SW2 Alps SKRK, U1 TLV75533PDBV, U101 RP2040, U103 W25Q16, U2 74HC4051, U3 74HC4051, U4 OPA350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

Commit message: couple extra bits
Other:
- board text added: "envious.design"
- board text removed: "When its all gone!?"
